File: pap/pap.kicad_pcb (KiCad board)
At the start: 2 copper layers, 16 parts, among them P1 CONN_01X02, P2 CONN_01X02, T1 TRANSFO_3PINS, U1 MC34063

Commit message: Misc. updates.
Parts:
- removed C5: 470uF, Capacitors_Elko_ThroughHole:Elko_vert_20x10mm_RM5
- added H1: ESP8266_07, papLib:ESP8266_07, F.Cu at (154.9, 97.8)
- added JP1: JUMPER3, Socket_Strips:Socket_Strip_Straight_1x03, F.Cu at (168.9, 90.2)
- added P3: CONN_01X03, Socket_Strips:Socket_Strip_Straight_1x03, F.Cu at (168.9, 106.7)
- added R4: 22k, Resistors_SMD:R_0805_HandSoldering, F.Cu at (160.0, 69.8)
- added R5: 13k, Resistors_SMD:R_0805_HandSoldering, F.Cu at (160.0, 76.2)
- added SW1: SW_PUSH, papLib:RST_SWITCH_SMD, F.Cu at (174.0, 101.6)
- added U2: MOC3020M, papLib:DIP-6__300, F.Cu at (121.9, 100.3)
- added U3: MC34063, papLib:DIP-8__300, F.Cu at (152.4, 71.1)
- C1: value 220pF -> 470uF; footprint Capacitors_ThroughHole:C_Disc_D3_P2.5 -> papLib:C_Radial_D8_L11.5_P3.5
- C2: value 100uF -> 220pF; footprint Capacitors_ThroughHole:C_Radial_D8_L11.5_P3.5 -> Capacitors_SMD:C_0805_HandSoldering
- C3: footprint Capacitors_ThroughHole:C_Radial_D6.3_L11.2_P2.5 -> Capacitors_SMD:c_elec_5x5.8
- C4: footprint Capacitors_ThroughHole:C_Radial_D8_L11.5_P3.5 -> Capacitors_SMD:c_elec_6.3x7.7
- D1: footprint Diodes_ThroughHole:Diode_DO-35_SOD27_Horizontal_RM10 -> Diodes_SMD:Diode-DO-214BA
- R1: value 1.8 -> 220; footprint Resistors_ThroughHole:Resistor_Horizontal_RM10mm -> Resistors_SMD:R_0805_HandSoldering
- R2: value 22k -> 220; footprint Resistors_ThroughHole:Resistor_Horizontal_RM10mm -> Resistors_SMD:R_0805_HandSoldering
- R3: value 13k -> 1.8
- U1: value MC34063 -> TRIAC; footprint Housings_DIP:DIP-8__300 -> Transistors_TO-220:TO-220_Neutral123_Vertical
- moved R1 123.4 mm to (115.6, 102.9), turned to 270 degrees
- moved P1 114.1 mm to (109.2, 96.5), turned to 90 degrees
- moved R3 101.5 mm to (144.8, 71.1), turned to 270 degrees
- moved C1 98.6 mm to (110.5, 82.5), turned to 180 degrees
- moved C3 89.4 mm to (166.4, 69.8), turned to 90 degrees
- moved U1 88.2 mm to (108.0, 102.9)
- moved D1 84.8 mm to (154.9, 82.5), turned to 180 degrees
- moved C4 81.7 mm to (147.3, 81.3), turned to 270 degrees
- moved L1 71.1 mm to (168.9, 81.3), turned to 270 degrees
- moved C2 66.2 mm to (154.9, 77.5)
- moved L2 52.0 mm to (154.9, 86.4)
- moved R2 50.4 mm to (174.0, 92.7), turned to 270 degrees
- moved P2 39.6 mm to (109.2, 68.6)
- moved BR1 38.1 mm to (133.3, 100.3)
- moved T1 30.2 mm to (129.5, 80.0)
Connections:
- C1 pad 1: Net-(C1-Pad1) -> /VCC
- C2 pad 1: /VCC -> Net-(C2-Pad1)
- D1 pad 2: /PIN2 -> Net-(D1-Pad2)
- L1 pad 1: /PIN2 -> Net-(D1-Pad2)
- P1 pad 1: /3.3v -> Net-(P1-Pad1)
- P1 pad 2: /GND -> Net-(P1-Pad2)
- R1 pad 1: /VCC -> Net-(R1-Pad1)
- R1 pad 2: /PIN7 -> Net-(P1-Pad2)
- R2 pad 1: Net-(R2-Pad1) -> /3.3v
- R2 pad 2: Net-(C3-Pad1) -> Net-(H1-Pad1)
- R3 pad 1: Net-(R2-Pad1) -> /VCC
- R3 pad 2: /GND -> /PIN7
- T1 pad 4: Net-(T1-Pad4) -> (no net)
- U1 pad 1: /PIN7 -> Net-(P1-Pad1)
- U1 pad 2: /PIN2 -> Net-(P1-Pad2)
- U1 pad 3: Net-(C1-Pad1) -> Net-(U1-Pad3)
Routing:
- net /VCC: track 0.00 -> 96.4 mm, vias 0 -> 2
- net Net-(H1-Pad7): track 0.00 -> 40.1 mm
- net /3.3v: track 0.00 -> 38.2 mm
- net Net-(C3-Pad1): track 0.00 -> 34.1 mm
- net Net-(D1-Pad2): track 0.00 -> 31.8 mm, vias 0 -> 2
- net Net-(BR1-Pad1): track 0.00 -> 29.8 mm
- net Net-(H1-Pad12): track 0.00 -> 28.8 mm
- net Net-(P1-Pad2): track 0.00 -> 27.3 mm
- net Net-(H1-Pad1): track 0.00 -> 26.8 mm, vias 0 -> 2
- net Net-(BR1-Pad2): track 0.00 -> 21.7 mm
- net /N: track 0.00 -> 17.2 mm
- net /PIN7: track 0.00 -> 14.5 mm
- net Net-(R4-Pad1): track 0.00 -> 13.5 mm
- net /L: track 0.00 -> 13.0 mm
- net Net-(H1-Pad15): track 0.00 -> 12.5 mm
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- added copper zone on B.Cu, net /GND
- added copper zone on F.Cu, net /GND
Other:
- net class Default: trace_width 0.25 -> 0.5; via_dia 0.6 -> 1.82; via_drill 0.4 -> 0.86
- rule trace_min: 0.2 -> 0.5
- rule via_min_drill: 0.3 -> 0.86
- rule via_min_size: 0.4 -> 1.82
