File: pap/pap.sch (KiCad schematic (older format))
At the start: 24 parts, among them P2 CONN_01X02, P3 CONN_01X02, P4 CONN_01X03, SW1 SW_PUSH, T1 TRANSFO_3PINS, U1 MC34063, U2 TRIAC, U3 MOC3023M

Commit message: Misc. updates.
Parts:
- removed C2: 100uF, Capacitors_Elko_ThroughHole:Elko_vert_11.5x8mm_RM3.5, symbol CP
- removed U1: MC34063, Housings_DIP:DIP-8__300, symbol MC34063
- removed U3: MOC3023M, DIP-6, symbol MOC3023M
- added U2: MOC3020M, DIP-6, symbol MOC3020M_MOD
- added U3: MC34063, symbol MC34063
- renumbered C5 to C1, C1 to C2, P3 to P1, P4 to P3, R4 to R1, R5 to R2, R1 to R3, R2 to R4, R3 to R5, U2 to U1
Connections:
- net GND: now also R5.1, U2.2, U3.4 (GND); no longer R5.2
- net PIN7: now also U3.1 (Sw_Coll), U3.7 (I_Sense), U3.8 (Drv_Coll)
- net VCC: now also U3.6 (VCC)
- net at C2.1: now also U3.3 (Tim_Cap)
- net at R4.1: now also R5.2, U3.5 (V_Sense); no longer R5.1
- net at H1.7 (GPIO13): now also U2.1
- net at U1.3: now also U2.4
- net at R1.1: now also U2.6
- net PIN2: no longer names the net of D1.2 (K), L1.1
- net PIN2: now also U3.2 (Sw_Emit)
Other:
- moved on the sheet: BR1, C1, C2, C3, C4, D1, H1, JP1, L1, L2, P1, P2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
